Commit message: [mini_quadrotor] Change default configuration to tilt-rotor model

File: robots/mini_quadrotor/urdf/robot.urdf.xacro (robot description, xacro)
@@ -6,7 +6,8 @@
   <thrust_link name="thrust" />
   <!-- kinematics [m] -->
-  <xacro:property name="rotor_x" value="0.070" />
-  <xacro:property name="rotor_y" value="0.086" />
-  <xacro:property name="rotor_z" value="0.026" />
+  <xacro:property name="rotor_x" value="0.117" />
+  <xacro:property name="rotor_y" value="0.109" />
+  <xacro:property name="rotor_z" value="0.036" />
+  <xacro:property name="rotor_tilt" value="${pi/9}" />
   <!-- dynamics -->
   <m_f_rate value="-0.011" /> <!-- drag torque rate -->
@@ -37,10 +38,10 @@
     </link>
   </xacro:macro>
-  <xacro:macro name="propeller_module" params="id x y z direction">
+  <xacro:macro name="propeller_module" params="id x y z direction tilt">
     <joint name="rotor${id}" type="continuous">
       <limit effort="100.0" lower="${min_force}" upper="${max_force}" velocity="0.5"/>
       <parent link="main_body"/>
       <child link="thrust${id}"/>
-      <origin rpy="0 0 0" xyz="${x} ${y} ${z}"/>
+      <origin rpy="${tilt} 0 ${-1 * direction * pi/4}" xyz="${x} ${y} ${z}"/>
       <axis xyz="0 0 ${direction}"/>
     </joint>
@@ -48,5 +49,5 @@
       <!-- visual & collisiont -->
       <inertial>
-        <origin xyz="0 0 0" rpy="0 0 0"/>
+        <origin xyz="0 0 0" rpy="${direction * 20 / pi} 0 0"/>
         <mass value="0.0091"/>
         <inertia
@@ -96,10 +97,10 @@
   <link name="main_body">
     <inertial>
-      <mass value = "0.432" />
-      <origin xyz="0 0 0.017" rpy="0 0 0"/>
+      <mass value = "0.546" />
+      <origin xyz="0 0 0.012" rpy="0 0 0"/>
       <inertia
-          ixx="0.0021" ixy="0" ixz="0"
-          iyy="0.0015" iyz="0"
-          izz="0.0032"/>
+          ixx="0.0045" ixy="0" ixz="0"
+          iyy="0.0045" iyz="0"
+          izz="0.0082"/>
     </inertial>
     <visual>
@@ -112,5 +113,5 @@
       <origin rpy="0 0 0" xyz="0 0 0"/>
       <geometry>
-        <box size="0.28 0.28 0.072" />
+        <box size="0.28 0.28 0.168" />
       </geometry>
     </collision>
@@ -127,43 +128,43 @@
     </inertial>
   </xacro:extra_module>
-  <!-- front realsense t265 -->
-  <xacro:extra_module name = "realsense_t265" parent = "main_body" visible = "1" scale= "1"
-                      model_url = "package://mini_quadrotor/urdf/mesh/realSense_t265.STL">
-    <origin xyz="0.1095 0.00775 0.0125" rpy="0 0 0"/>
-    <inertial>
-      <mass value = "0.07" />
-      <origin xyz="-0.007 -0.007 0" rpy="0 0 0"/>
-      <inertia
-          ixx="0.0" ixy="0.0" ixz="0.0"
-          iyy="0.0001" iyz="0.0"
-          izz="0.0001"/>
-    </inertial>
-  </xacro:extra_module>
-  <!-- pose frame for realsense t265 -->
-  <xacro:extra_module name = "realsense_pose_frame" parent = "realsense_t265" visible = "0" >
-    <origin xyz="-0.005 0.0 0.0" rpy="0 0 0"/>
-    <inertial>
-      <mass value = "0.0" />
-      <origin xyz="0 0 0" rpy="0 0 0"/>
-      <inertia
-          ixx="0.0" ixy="0.0" ixz="0.0"
-          iyy="0.0" iyz="0.0" izz="0.0"/>
-    </inertial>
-  </xacro:extra_module>
-  <!-- battery -->
-  <xacro:extra_module name = "battery" parent = "main_body" visible = "1" model_url = "package://mini_quadrotor/urdf/mesh/turnigy_3S_2200mAh.dae" >
-    <origin xyz="0.0105 0 -0.012" rpy="0 0 0"/>
-    <inertial>
-      <mass value = "0.188" />
-      <origin xyz="0 0 0" rpy="0 0 0"/>
-      <inertia
-          ixx="0.0" ixy="0.0" ixz="0.0"
-          iyy="0.0002" iyz="0.0" izz="0.0002"/>
-    </inertial>
-  </xacro:extra_module>
+  <!-- <!-\- front realsense t265 -\-> -->
+  <!-- <xacro:extra_module name = "realsense_t265" parent = "main_body" visible = "1" scale= "1" -->
+  <!--                     model_url = "package://mini_quadrotor/urdf/mesh/realSense_t265.STL"> -->
+  <!--   <origin xyz="0.1095 0.00775 0.0125" rpy="0 0 0"/> -->
+  <!--   <inertial> -->
+  <!--     <mass value = "0.07" /> -->
+  <!--     <origin xyz="-0.007 -0.007 0" rpy="0 0 0"/> -->
+  <!--     <inertia -->
+  <!--         ixx="0.0" ixy="0.0" ixz="0.0" -->
+  <!--         iyy="0.0001" iyz="0.0" -->
+  <!--         izz="0.0001"/> -->
+  <!--   </inertial> -->
+  <!-- </xacro:extra_module> -->
+  <!-- <!-\- pose frame for realsense t265 -\-> -->
+  <!-- <xacro:extra_module name = "realsense_pose_frame" parent = "realsense_t265" visible = "0" > -->
+  <!--   <origin xyz="-0.005 0.0 0.0" rpy="0 0 0"/> -->
+  <!--   <inertial> -->
+  <!--     <mass value = "0.0" /> -->
+  <!--     <origin xyz="0 0 0" rpy="0 0 0"/> -->
+  <!--     <inertia -->
+  <!--         ixx="0.0" ixy="0.0" ixz="0.0" -->
+  <!--         iyy="0.0" iyz="0.0" izz="0.0"/> -->
+  <!--   </inertial> -->
+  <!-- </xacro:extra_module> -->
+  <!-- <!-\- battery -\-> -->
+  <!-- <xacro:extra_module name = "battery" parent = "main_body" visible = "1" model_url = "package://mini_quadrotor/urdf/mesh/turnigy_3S_2200mAh.dae" > -->
+  <!--   <origin xyz="0.0105 0 -0.012" rpy="0 0 0"/> -->
+  <!--   <inertial> -->
+  <!--     <mass value = "0.188" /> -->
+  <!--     <origin xyz="0 0 0" rpy="0 0 0"/> -->
+  <!--     <inertia -->
+  <!--         ixx="0.0" ixy="0.0" ixz="0.0" -->
+  <!--         iyy="0.0002" iyz="0.0" izz="0.0002"/> -->
+  <!--   </inertial> -->
+  <!-- </xacro:extra_module> -->
   <!-- propellers -->
-  <xacro:propeller_module id = "1" x = "${-rotor_x}" y = "${-rotor_y}" z = "${rotor_z}" direction = "-1" />
-  <xacro:propeller_module id = "2" x = "${rotor_x}" y = "${-rotor_y}" z = "${rotor_z}" direction = "1" />
-  <xacro:propeller_module id = "3" x = "${rotor_x}" y = "${rotor_y}" z = "${rotor_z}" direction = "-1" />
-  <xacro:propeller_module id = "4" x = "${-rotor_x}" y = "${rotor_y}" z = "${rotor_z}"  direction = "1" />
+  <xacro:propeller_module id = "1" x = "${-rotor_x}" y = "${-rotor_y}" z = "${rotor_z}" direction = "-1" tilt = "${-rotor_tilt}"/>
+  <xacro:propeller_module id = "2" x = "${rotor_x}" y = "${-rotor_y}" z = "${rotor_z}" direction = "1" tilt = "${-rotor_tilt}"/>
+  <xacro:propeller_module id = "3" x = "${rotor_x}" y = "${rotor_y}" z = "${rotor_z}" direction = "-1" tilt = "${rotor_tilt}"/>
+  <xacro:propeller_module id = "4" x = "${-rotor_x}" y = "${rotor_y}" z = "${rotor_z}"  direction = "1" tilt = "${rotor_tilt}"/>
 </robot>

Commit message: [mini_quadrotor] fixed urdf to match the real aircraft

File: robots/mini_quadrotor/urdf/robot.urdf.xacro (robot description, xacro)
@@ -43,5 +43,5 @@
       <parent link="main_body"/>
       <child link="thrust${id}"/>
-      <origin rpy="${tilt} 0 ${-1 * direction * pi/4}" xyz="${x} ${y} ${z}"/>
+      <origin rpy="${tilt} 0 ${direction * pi/4}" xyz="${x} ${y} ${z}"/>
       <axis xyz="0 0 ${direction}"/>
     </joint>
@@ -164,7 +164,7 @@
   <!-- </xacro:extra_module> -->
   <!-- propellers -->
-  <xacro:propeller_module id = "1" x = "${-rotor_x}" y = "${-rotor_y}" z = "${rotor_z}" direction = "-1" tilt = "${-rotor_tilt}"/>
-  <xacro:propeller_module id = "2" x = "${rotor_x}" y = "${-rotor_y}" z = "${rotor_z}" direction = "1" tilt = "${-rotor_tilt}"/>
-  <xacro:propeller_module id = "3" x = "${rotor_x}" y = "${rotor_y}" z = "${rotor_z}" direction = "-1" tilt = "${rotor_tilt}"/>
-  <xacro:propeller_module id = "4" x = "${-rotor_x}" y = "${rotor_y}" z = "${rotor_z}"  direction = "1" tilt = "${rotor_tilt}"/>
+  <xacro:propeller_module id = "1" x = "${-rotor_x}" y = "${-rotor_y}" z = "${rotor_z}" direction = "1" tilt = "${-rotor_tilt}"/>
+  <xacro:propeller_module id = "2" x = "${rotor_x}" y = "${-rotor_y}" z = "${rotor_z}" direction = "-1" tilt = "${-rotor_tilt}"/>
+  <xacro:propeller_module id = "3" x = "${rotor_x}" y = "${rotor_y}" z = "${rotor_z}" direction = "1" tilt = "${rotor_tilt}"/>
+  <xacro:propeller_module id = "4" x = "${-rotor_x}" y = "${rotor_y}" z = "${rotor_z}"  direction = "-1" tilt = "${rotor_tilt}"/>
 </robot>
