Commit message: [mini_quadrotor] Update mass and inertia

File: robots/mini_quadrotor/urdf/dual/robot.urdf.xacro (robot description, xacro)
@@ -99,10 +99,10 @@
   <link name="main_body1">
     <inertial>
-      <mass value = "0.546" />
+          <mass value = "0.509" />
       <origin xyz="0 0 0.012" rpy="0 0 0"/>
       <inertia
-          ixx="0.0045" ixy="0" ixz="0"
-          iyy="0.0045" iyz="0"
-          izz="0.0082"/>
+          ixx="0.0038" ixy="0.0000043" ixz="0.0000086"
+          iyy="0.0042" iyz="-0.0000053"
+          izz="0.0072"/>
     </inertial>
     <visual>
@@ -138,19 +138,22 @@
       </visual>
   </link>
-  <joint name="flex_joint1" type="fixed">
+  <joint name="flex_joint1" type="revolute">
+  <!-- <joint name="flex_joint1" type="fixed"> -->
     <parent link="main_body1"/>
     <child link="flex_link"/>
     <origin rpy="0 0 0" xyz="0 0 ${-flex_joint_offset_z}"/>
     <axis xyz="1 0 0"/>
+    <limit effort="0.001" lower="${-pi/2}" upper="${pi/2}" velocity="1"/>
+    <dynamics damping="0.1" friction="0.0"/>
   </joint>
   <!-- main_body2 -->
   <link name="main_body2">
     <inertial>
-      <mass value = "0.546" />
+          <mass value = "0.509" />
       <origin xyz="0 0 0.012" rpy="0 0 0"/>
       <inertia
-          ixx="0.0045" ixy="0" ixz="0"
-          iyy="0.0045" iyz="0"
-          izz="0.0082"/>
+          ixx="0.0038" ixy="0.0000043" ixz="0.0000086"
+          iyy="0.0042" iyz="-0.0000053"
+          izz="0.0072"/>
     </inertial>
     <visual>

File: robots/mini_quadrotor/urdf/single/robot.urdf.xacro (robot description, xacro)
@@ -97,10 +97,10 @@
   <link name="main_body">
     <inertial>
-      <mass value = "0.546" />
+      <mass value = "0.509" />
       <origin xyz="0 0 0.012" rpy="0 0 0"/>
       <inertia
-          ixx="0.0045" ixy="0" ixz="0"
-          iyy="0.0045" iyz="0"
-          izz="0.0082"/>
+          ixx="0.0038" ixy="0.0000043" ixz="0.0000086"
+          iyy="0.0042" iyz="-0.0000053"
+          izz="0.0072"/>
     </inertial>
     <visual>

Commit message: [mini_quadrotor] Fix bug : urdf model of eight rotor model

File: robots/mini_quadrotor/urdf/dual/robot.urdf.xacro (robot description, xacro)
@@ -45,5 +45,5 @@
       <parent link="${par_link}"/>
       <child link="thrust${id}"/>
-      <origin rpy="${tilt} 0 ${-1 * direction * pi/4}" xyz="${x} ${y} ${z}"/>
+      <origin rpy="${tilt} 0 ${direction * pi/4}" xyz="${x} ${y} ${z}"/>
       <axis xyz="0 0 ${direction}"/>
     </joint>
@@ -223,11 +223,11 @@
   <!-- </xacro:extra_module> -->
   <!-- propellers -->
-  <xacro:propeller_module id = "1" x = "${-rotor_x}" y = "${-rotor_y}" z = "${rotor_z}" direction = "-1" tilt = "${-rotor_tilt}" par_link = "main_body1"/>
-  <xacro:propeller_module id = "2" x = "${rotor_x}" y = "${-rotor_y}" z = "${rotor_z}" direction = "1" tilt = "${-rotor_tilt}" par_link = "main_body1"/>
-  <xacro:propeller_module id = "3" x = "${rotor_x}" y = "${rotor_y}" z = "${rotor_z}" direction = "-1" tilt = "${rotor_tilt}" par_link = "main_body1"/>
-  <xacro:propeller_module id = "4" x = "${-rotor_x}" y = "${rotor_y}" z = "${rotor_z}"  direction = "1" tilt = "${rotor_tilt}" par_link = "main_body1"/>
-  <xacro:propeller_module id = "5" x = "${-rotor_x}" y = "${-rotor_y}" z = "${rotor_z}" direction = "-1" tilt = "${-rotor_tilt}" par_link = "main_body2"/>
-  <xacro:propeller_module id = "6" x = "${rotor_x}" y = "${-rotor_y}" z = "${rotor_z}" direction = "1" tilt = "${-rotor_tilt}" par_link = "main_body2"/>
-  <xacro:propeller_module id = "7" x = "${rotor_x}" y = "${rotor_y}" z = "${rotor_z}" direction = "-1" tilt = "${rotor_tilt}" par_link = "main_body2"/>
-  <xacro:propeller_module id = "8" x = "${-rotor_x}" y = "${rotor_y}" z = "${rotor_z}"  direction = "1" tilt = "${rotor_tilt}" par_link = "main_body2"/>
+  <xacro:propeller_module id = "1" x = "${-rotor_x}" y = "${-rotor_y}" z = "${rotor_z}" direction = "1" tilt = "${-rotor_tilt}" par_link = "main_body1"/>
+  <xacro:propeller_module id = "2" x = "${rotor_x}" y = "${-rotor_y}" z = "${rotor_z}" direction = "-1" tilt = "${-rotor_tilt}" par_link = "main_body1"/>
+  <xacro:propeller_module id = "3" x = "${rotor_x}" y = "${rotor_y}" z = "${rotor_z}" direction = "1" tilt = "${rotor_tilt}" par_link = "main_body1"/>
+  <xacro:propeller_module id = "4" x = "${-rotor_x}" y = "${rotor_y}" z = "${rotor_z}"  direction = "-1" tilt = "${rotor_tilt}" par_link = "main_body1"/>
+  <xacro:propeller_module id = "5" x = "${-rotor_x}" y = "${-rotor_y}" z = "${rotor_z}" direction = "1" tilt = "${-rotor_tilt}" par_link = "main_body2"/>
+  <xacro:propeller_module id = "6" x = "${rotor_x}" y = "${-rotor_y}" z = "${rotor_z}" direction = "-1" tilt = "${-rotor_tilt}" par_link = "main_body2"/>
+  <xacro:propeller_module id = "7" x = "${rotor_x}" y = "${rotor_y}" z = "${rotor_z}" direction = "1" tilt = "${rotor_tilt}" par_link = "main_body2"/>
+  <xacro:propeller_module id = "8" x = "${-rotor_x}" y = "${rotor_y}" z = "${rotor_z}"  direction = "-1" tilt = "${rotor_tilt}" par_link = "main_body2"/>
 </robot>
