Commit message: fix(urdf): corrected LiDAR frame orientation

File: robots/gimbalrotor/urdf/ynltilt/gimbalrotor.urdf.xacro (robot description, xacro)
@@ -241,5 +241,5 @@
   </xacro:macro>
   <xacro:extra_module name = "lidar_imu" parent = "base_link" visible = "0" > <!-- should be IMU frame -->
-    <origin xyz="${0.0} ${0.0} ${0.145}" rpy="0 0 ${pi/2.0}"/> <!-- TODO: the true pos -->
+    <origin xyz="${0.0} ${0.0} ${0.145}" rpy="0 0 ${-pi/2.0}"/> <!-- TODO: the true pos -->
     <inertial>
       <mass value = "00" />
